File: Hardware/LampeSolaire/LampeSolaire.sch (KiCad schematic (older format))
At the start: 124 parts, among them K1 RELAIS_DPDT, P1 1V8, P2 3V5, P3 3V5, T1 SI2333, T2 FDN337, T3 FDN337, T4 FDN337, T5 FDN337, U1 MCP73832, U2 MCP121, U3 NCP114ASN330T1G, U4 3V3 to 5V, U5 RF_RECEIVER, U6 PIC16F1827, U7 MCP6001R, U8 74LV00, X1 ICSP, X13 STOCK, X14 STOCK, X15 STOCK, X17 STOCK_1, X18 SOLAR_CELL, X2 PHOTO_RESISTOR, X3 WATER_SENSOR, X4 WATER_SENSOR, X5 LAMP, X6 STOCK_1, X8 BUZZER

Commit message: Version 4
Nouveau PCB, modifications diverses au schéma
Parts:
- removed C10, C9: 100nF, Capacitors_SMD:C_1206_HandSoldering, symbol MyLib:CAPA
- removed C7: 4.7uF, MyLib:CP_Radial_D5.0mm_P2.00mm, symbol MyLib:CAPA_P
- removed R11: 110k, MyLib:R_0805_HandSoldering, symbol MyLib:R
- removed R12, R13, R17: 100k, MyLib:R_0805_HandSoldering, symbol MyLib:R
- removed R16: 150k, MyLib:R_0805_HandSoldering, symbol MyLib:R
- removed TP1, TP11, TP12, TP14, TP15, TP17, TP18, TP19, TP2, TP20, TP21, TP22, TP23, TP24, TP25, TP26, TP27, TP28, TP29, TP30, TP36, TP38, TP39, TP4, TP40, TP41, TP42, TP43, TP44, TP45, TP49, TP5, TP50, TP51, TP6, TP7, TP9: TestPoint, MyLib:Measurement_Point_Round-SMD-Pad_Small, symbol MyLib:TestPoint
- removed TP35: TestPoint_8, MyLib:Measurement_Point_Round-TH_Small_x8, symbol MyLib:TestPoint_8
- removed U4: 3V3 to 5V, MyLib:DC_DC, symbol MyLib:DC-DC
- removed U7: MCP6001R, MyLib:SOT-23-5_HandSoldering, symbol MyLib:MCP6001R
- removed U8: 74LV00, MyLib:SOIC-14, symbol MyLib:74xx00
- removed W10, W11, W12, W13, W14, W15, W16, W17, W18, W20, W21, W22, W4, W7, W8, W9: TEST_2P, MyLib:Pin_Header_Straight_1x02_Pitch2.54mm, symbol MyLib:TEST_2P
- removed X13, X14, X15: STOCK, MyLib:Pin_Header_Straight_1x02_Pitch2.54mm, symbol MyLib:CONN_01X02
- removed X5: LAMP, MyLib:Pin_Header_Straight_1x02_Pitch2.54mm, symbol MyLib:CONN_01X02
- added R4: 100k, MyLib:R_0805_HandSoldering, symbol MyLib:R
- added T2: SI2333, MyLib:SOT-23_Handsoldering, symbol ShockAccel:MOSFET-P
- added T3: FDN337, MyLib:SOT-23_Handsoldering, symbol MyLib:MOSFET-N
- added TP5: TestPoint_8, MyLib:Measurement_Point_Round-TH_Small, symbol MyLib:TestPoint_8
- added U6: 74xx00, MyLib:SOIC-14, symbol MyLib:74xx00
- F1: footprint MyLib:FuseHolder_Schurter -> Fuse_Holders_and_Fuses:Fuse_SMD1206_HandSoldering
- R5: renamed from R4; value 4k7 -> 1k
- R6: renamed from R5; value 4k7 -> 1k
- R7: renamed from R6; value 4k7 -> 1k
- R8: renamed from R7; value 4k7 -> 1k
- TP1: renamed from TP31; footprint MyLib:Measurement_Point_Round-TH_Small_x8 -> MyLib:Measurement_Point_Round-TH_Small
- TP2: renamed from TP32; footprint MyLib:Measurement_Point_Round-TH_Small_x8 -> MyLib:Measurement_Point_Round-TH_Small
- TP3: renamed from TP33; footprint MyLib:Measurement_Point_Round-TH_Small_x8 -> MyLib:Measurement_Point_Round-TH_Small
- TP4: renamed from TP34; footprint MyLib:Measurement_Point_Round-TH_Small_x8 -> MyLib:Measurement_Point_Round-TH_Small
- renumbered C8 to C6, R19 to R10, R9 to R11, R10 to R12, R14 to R13, R15 to R14, R8 to R9, T2 to T4, T4 to T5, T3 to T6, T5 to T7, TP3 to TP6, U5 to U4, U6 to U5, W3 to W1, W1 to W2, W2 to W3, W19 to W4, W23 to W5, X18 to X1, X1 to X2, X6 to X3, X8 to X4, X2 to X5, X3 to X6, X4 to X7, X17 to X8
Connections:
- net labels added: VBAT_0
- net labels removed: +5V, 1V9, LAMP
- wire segments 323 -> 242
- no-connect marks 3 -> 5
Other:
- note added: "Max power : 750mW\nDo not set those\ntrimmer above 8 ohm\nSet the current\nto 300mA"
- note added: "R4..7 :\n4x 1k"
- note removed: "Max power : 750mW\nDo not set those trimmer above 8 ohm\nSet the current to 300mA"
- note removed: "R4..7 :\n4x 4k7"

Commit message: Updated rf module
Uses now transceiver 860MHz
Parts:
- removed R11: 1M, MyLib:R_0805_HandSoldering, symbol MyLib:R
- removed R5, R6, R7, R8: 1k, MyLib:R_0805_HandSoldering, symbol MyLib:R
- removed R9: 4k7, MyLib:R_0805_HandSoldering, symbol MyLib:R
- removed U4: RF_RECEIVER, MyLib:RF_RECEIVER, symbol MyLib:RF_RECEIVER
- removed X3, X8: STOCK_1, MyLib:Pin_Header_Straight_1x01_Pitch2.54mm, symbol MyLib:CONN_01X01
- removed X5: PHOTO_RESISTOR, MyLib:Pin_Header_Straight_1x02_Pitch2.54mm, symbol MyLib:CONN_01X02
- removed X7: WATER_SENSOR, MyLib:Pin_Header_Straight_1x02_Pitch2.54mm, symbol MyLib:CONN_01X02
- added C7: 4.7uF, Capacitors_SMD:C_1206_HandSoldering, symbol 0EsseivaN_Lib:CAPA
- added C8: 100nF, Capacitors_SMD:C_1206_HandSoldering, symbol 0EsseivaN_Lib:CAPA
- added P4: 2V, 0EsseivaN_Lib:D_0603_HandSoldering, symbol 0EsseivaN_Lib:LED
- added R5, R8, R9: 1K, 0EsseivaN_Lib:R_0805_HandSoldering, symbol 0EsseivaN_Lib:R
- added R6: 330R, 0EsseivaN_Lib:R_0805_HandSoldering, symbol 0EsseivaN_Lib:R
- added R7: 100kR, 0EsseivaN_Lib:R_0805_HandSoldering, symbol 0EsseivaN_Lib:R
- added U4: MRF89XAM8A, symbol 0EsseivaN_Lib:MRF89XAM8A
- C1, C2: footprint MyLib:CP_Radial_D5.0mm_P2.00mm -> 0EsseivaN_Lib:CP_Radial_D5.0mm_P2.00mm; symbol MyLib:CAPA_P -> 0EsseivaN_Lib:CAPA_P
- C3, C4, C5, C6: symbol MyLib:CAPA -> 0EsseivaN_Lib:CAPA
- F1: symbol MyLib:Fuse -> 0EsseivaN_Lib:Fuse
- K1: footprint MyLib:Relay -> 0EsseivaN_Lib:Relay; symbol MyLib:RELAIS_DPDT -> 0EsseivaN_Lib:RELAIS_DPDT
- P1: footprint MyLib:LED_D3.0mm -> 0EsseivaN_Lib:LED_D3.0mm; symbol LampeSolaire-rescue:LED-RESCUE-LampeSolaire -> 0EsseivaN_Lib:LED
- P2, P3: footprint MyLib:Pin_Header_Straight_1x02_Pitch2.54mm -> 0EsseivaN_Lib:Pin_Header_Straight_1x02_Pitch2.54mm; symbol LampeSolaire-rescue:LED-RESCUE-LampeSolaire -> 0EsseivaN_Lib:LED
- R1, R10, R12, R3, R4: footprint MyLib:R_0805_HandSoldering -> 0EsseivaN_Lib:R_0805_HandSoldering; symbol MyLib:R -> 0EsseivaN_Lib:R
- R13, R14: footprint MyLib:Potentiometer_Trimmer_Bourns_3006P -> 0EsseivaN_Lib:Potentiometer_Trimmer_Bourns_3006P; symbol MyLib:Trimmer -> 0EsseivaN_Lib:Trimmer
- R2: footprint MyLib:T93YB -> 0EsseivaN_Lib:T93YB; symbol EMF-Symbols:TRIMMER -> 0EsseivaN_Lib:TRIMMER
- SC1: footprint MyLib:Pin_Header_Straight_1x02_Pitch2.54mm -> 0EsseivaN_Lib:Pin_Header_Straight_1x02_Pitch2.54mm; symbol MyLib:Solar_Cells -> 0EsseivaN_Lib:Solar_Cells
- T1, T2: footprint MyLib:SOT-23_Handsoldering -> 0EsseivaN_Lib:SOT-23_Handsoldering; symbol ShockAccel:MOSFET-P -> 0EsseivaN_Lib:MOSFET-P
- T3, T4, T5, T6, T7: footprint MyLib:SOT-23_Handsoldering -> 0EsseivaN_Lib:SOT-23_Handsoldering; symbol MyLib:MOSFET-N -> 0EsseivaN_Lib:MOSFET-N
- TP1, TP2, TP3, TP4, TP5: footprint MyLib:Measurement_Point_Round-TH_Small -> 0EsseivaN_Lib:Measurement_Point_Round-TH_Small; symbol MyLib:TestPoint_8 -> 0EsseivaN_Lib:TestPoint_8
- TP6: footprint MyLib:Measurement_Point_Round-SMD-Pad_Small -> 0EsseivaN_Lib:Measurement_Point_Round-SMD-Pad_Small; symbol MyLib:TestPoint -> 0EsseivaN_Lib:TestPoint
- U1: footprint MyLib:SOT-23-5_HandSoldering -> 0EsseivaN_Lib:SOT-23-5_HandSoldering; symbol ShockAccel:MCP73832 -> 0EsseivaN_Lib:MCP73832
- U2: footprint ShockAccel:SOT-23_Handsoldering -> 0EsseivaN_Lib:SOT-23_Handsoldering; symbol ShockAccel:MCP121 -> 0EsseivaN_Lib:MCP121
- U3: footprint MyLib:TSOP-5 -> 0EsseivaN_Lib:TSOP-5; symbol MyLib:MIC5504 -> 0EsseivaN_Lib:MIC5504
- U5: footprint MyLib:DIP-18 -> 0EsseivaN_Lib:DIP-18; symbol LampeSolaire-rescue:PIC16F1827 -> 0EsseivaN_Lib:PIC16F1827
- U6: footprint MyLib:SOIC-14 -> 0EsseivaN_Lib:SOIC-14; symbol MyLib:74xx00 -> 0EsseivaN_Lib:74xx00
- V1: footprint MyLib:Pin_Header_Straight_1x02_Pitch2.54mm -> 0EsseivaN_Lib:Pin_Header_Straight_1x02_Pitch2.54mm; symbol ShockAccel:LiPo -> 0EsseivaN_Lib:LiPo
- W1, W2, W3, W4, W5, W6: footprint MyLib:Pin_Header_Straight_1x02_Pitch2.54mm -> 0EsseivaN_Lib:Pin_Header_Straight_1x02_Pitch2.54mm; symbol MyLib:TEST_2P -> 0EsseivaN_Lib:TEST_2P
- X1, X4, X6: footprint MyLib:Pin_Header_Straight_1x02_Pitch2.54mm -> 0EsseivaN_Lib:Pin_Header_Straight_1x02_Pitch2.54mm; symbol MyLib:CONN_01X02 -> 0EsseivaN_Lib:CONN_01X02
- X2: footprint MyLib:Pin_Header_Angled_1x06_Pitch2.54mm_reverse_invis -> 0EsseivaN_Lib:Pin_Header_Angled_1x06_Pitch2.54mm_reverse_invis; symbol MyLib:CONN_01X05 -> 0EsseivaN_Lib:CONN_01X05
Connections:
- net labels added: BUZZER, IRQ0, IRQ1, LED, MISO, MOSI, SCK, WATER, ~CSCON, ~CSDATA
- net labels removed: INT
- wire segments 242 -> 282
Other:
- note removed: "R4..7 :\n4x 1k"

Commit message: Schematic v5 and PCB v5.1
Parts:
- removed R13, R14: 10, 0EsseivaN_Lib:Potentiometer_Trimmer_Bourns_3006P, symbol 0EsseivaN_Lib:Trimmer
- removed R2: 100k, 0EsseivaN_Lib:T93YB, symbol 0EsseivaN_Lib:TRIMMER
- removed TP1, TP2, TP3, TP4, TP5: TestPoint_8, 0EsseivaN_Lib:Measurement_Point_Round-TH_Small, symbol 0EsseivaN_Lib:TestPoint_8
- removed TP6: TestPoint, 0EsseivaN_Lib:Measurement_Point_Round-SMD-Pad_Small, symbol 0EsseivaN_Lib:TestPoint
- removed W1, W6: TEST_2P, 0EsseivaN_Lib:Pin_Header_Straight_1x02_Pitch2.54mm, symbol 0EsseivaN_Lib:TEST_2P
- added R11, R13: 6, Resistors_SMD:R_1206_HandSoldering, symbol 0EsseivaN_Lib:R
- added R2: 3k9, 0EsseivaN_Lib:R_0805_HandSoldering, symbol 0EsseivaN_Lib:R
- C7: footprint Capacitors_SMD:C_1206_HandSoldering -> 0EsseivaN_Lib:CP_Radial_D5.0mm_P2.00mm
- P2, P3, SC1, X1, X4, X6: footprint 0EsseivaN_Lib:Pin_Header_Straight_1x02_Pitch2.54mm -> 0EsseivaN_Lib:CH_2P
- R7: value 100kR -> 100k
- U4: footprint (none) -> 0EsseivaN_Lib:MRF89XAM8A
- U5: footprint 0EsseivaN_Lib:DIP-18 -> Housings_SSOP:SSOP-20_5.3x7.2mm_Pitch0.65mm
- V1: footprint 0EsseivaN_Lib:Pin_Header_Straight_1x02_Pitch2.54mm -> 0EsseivaN_Lib:CH_3P
- X2: footprint 0EsseivaN_Lib:Pin_Header_Angled_1x06_Pitch2.54mm_reverse_invis -> 0EsseivaN_Lib:Pin_Header_Angled_1x06_Pitch2.54mm
Connections:
- net labels added: RESET_RF
- wire segments 282 -> 262

Commit message: To remap because of error on ssop mcu
Parts:
- U5: symbol 0EsseivaN_Lib:PIC16F1827 -> 0EsseivaN_Lib:PIC16F1827_20
Connections:
- wire segments 262 -> 268
Changed lines of the file:
@@
 	2100 900  3200 900
 Wire Wire Line
-	5700 3000 5700 3300
+	5700 3000 5700 3200
 Wire Wire Line
 	1300 900  1400 900
@@
 $EndComp
 $Comp
-L 0EsseivaN_Lib:PIC16F1827 U5
+L 0EsseivaN_Lib:PIC16F1827_20 U5
 U 1 1 5B65DEBF
 P 5700 4300
@@
 Text Label 1050 4050 2    60   ~ 0
 RESET_RF
+Wire Wire Line
+	5600 3300 5600 3200
+Wire Wire Line
+	5600 3200 5700 3200
+Connection ~ 5700 3200
+Wire Wire Line
+	5800 3300 5800 3200
+Wire Wire Line
+	5800 3200 5700 3200
+Wire Wire Line
+	5600 5300 5700 5300
+Connection ~ 5700 5300
+Wire Wire Line
+	5700 5300 5800 5300
 $EndSCHEMATC

Commit message: Remap complete
Commit before cleanup and size reducing
Parts:
- X2: footprint 0EsseivaN_Lib:Pin_Header_Angled_1x06_Pitch2.54mm -> 0EsseivaN_Lib:Pin_Header_Straight_1x06_Pitch2.54mm
Changed lines of the file:
@@
 Sheet 1 1
 Title "Lampe Solaire"
-Date "2019-04-23"
+Date "2019-04-26"
 Rev "5"
 Comp "EsseivaN"
@@
 F 0 "X2" H 717 3415 50  0000 C CNN
 F 1 "ICSP" H 717 3324 50  0000 C CNN
-F 2 "0EsseivaN_Lib:Pin_Header_Angled_1x06_Pitch2.54mm" H 800 2900 50  0001 C CNN
+F 2 "0EsseivaN_Lib:Pin_Header_Straight_1x06_Pitch2.54mm" H 800 2900 50  0001 C CNN
 F 3 "" H 800 2900 50  0000 C CNN
 	1    800  2900

Commit message: V5 Complete
Parts:
- P2, P3, SC1, X4, X6: footprint 0EsseivaN_Lib:CH_2P -> 0EsseivaN_Lib:CH_02P
- SC2: renamed from X1; footprint 0EsseivaN_Lib:CH_2P -> 0EsseivaN_Lib:CH_02P
- V1: footprint 0EsseivaN_Lib:CH_3P -> 0EsseivaN_Lib:CH_03P
Changed lines of the file:
@@
 F 0 "SC1" H 1408 1753 50  0000 L CNN
 F 1 "Solar_Cells" H 1400 1700 50  0001 L CNN
-F 2 "0EsseivaN_Lib:CH_2P" V 1300 1760 50  0001 C CNN
+F 2 "0EsseivaN_Lib:CH_02P" V 1300 1760 50  0001 C CNN
 F 3 "" V 1300 1760 50  0000 C CNN
 F 4 "5V" H 1408 1654 60  0000 L CNN "Voltage"
@@
 F 0 "P2" V 9547 6022 60  0000 R CNN
 F 1 "3V5" V 9653 6022 60  0000 R CNN
-F 2 "0EsseivaN_Lib:CH_2P" H 9600 6200 60  0001 C CNN
+F 2 "0EsseivaN_Lib:CH_02P" H 9600 6200 60  0001 C CNN
 F 3 "" H 9600 6200 60  0000 C CNN
 	1    9600 6200
@@
 F 0 "P3" V 9947 6278 60  0000 L CNN
 F 1 "3V5" V 10053 6278 60  0000 L CNN
-F 2 "0EsseivaN_Lib:CH_2P" H 10000 6200 60  0001 C CNN
+F 2 "0EsseivaN_Lib:CH_02P" H 10000 6200 60  0001 C CNN
 F 3 "" H 10000 6200 60  0000 C CNN
 	1    10000 6200
@@
 $EndComp
 $Comp
-L 0EsseivaN_Lib:CONN_01X02 X1
+L 0EsseivaN_Lib:CONN_01X02 SC2
 U 1 1 5B71F5E8
 P 800 1300
-F 0 "X1" H 878 1341 50  0000 L CNN
+F 0 "SC2" H 878 1341 50  0000 L CNN
 F 1 "SOLAR_CELL" H 878 1250 50  0000 L CNN
-F 2 "0EsseivaN_Lib:CH_2P" H 800 1250 50  0001 C CNN
+F 2 "0EsseivaN_Lib:CH_02P" H 800 1250 50  0001 C CNN
 F 3 "" H 800 1250 50  0000 C CNN
 	1    800  1300
@@
 F 0 "X4" H 4117 2715 50  0000 C CNN
 F 1 "BUZZER" H 4117 2624 50  0000 C CNN
-F 2 "0EsseivaN_Lib:CH_2P" H 4200 2350 50  0001 C CNN
+F 2 "0EsseivaN_Lib:CH_02P" H 4200 2350 50  0001 C CNN
 F 3 "" H 4200 2350 50  0000 C CNN
 	1    4200 2400
@@
 F 0 "V1" H 5450 1950 60  0000 C CNN
 F 1 "Li battery" H 5600 1850 60  0000 C CNN
-F 2 "0EsseivaN_Lib:CH_3P" H 5310 1750 60  0001 C CNN
+F 2 "0EsseivaN_Lib:CH_03P" H 5310 1750 60  0001 C CNN
 F 3 "" H 5310 1750 60  0001 C CNN
 F 4 "3V7" H 5500 1550 60  0000 C CNN "Voltage"
@@
 F 0 "X6" H 7628 2691 50  0000 L CNN
 F 1 "WATER_SENSOR" H 7628 2600 50  0000 L CNN
-F 2 "0EsseivaN_Lib:CH_2P" H 7550 2600 50  0001 C CNN
+F 2 "0EsseivaN_Lib:CH_02P" H 7550 2600 50  0001 C CNN
 F 3 "" H 7550 2600 50  0000 C CNN
 	1    7550 2650

Commit message: Update for next version
Parts:
- removed K1: RELAIS_DPDT, 0EsseivaN_Lib:Relay, symbol 0EsseivaN_Lib:RELAIS_DPDT
- removed SC2: SOLAR_CELL, 0EsseivaN_Lib:CH_02P, symbol 0EsseivaN_Lib:CONN_01X02
- removed T4, T5, T6, T7: FDN337, 0EsseivaN_Lib:SOT-23_Handsoldering, symbol 0EsseivaN_Lib:MOSFET-N
- removed U6: 74xx00, 0EsseivaN_Lib:SOIC-14, symbol 0EsseivaN_Lib:74xx00
- added C10: 4.7uF, 0EsseivaN_Lib:C_0805_HandSoldering, symbol 0EsseivaN_Lib:CAPA
- added C11, C9: 100nF, Capacitors_SMD:C_1206_HandSoldering, symbol 0EsseivaN_Lib:CAPA
- added U6: MCP9700, 0EsseivaN_Lib:SOT-23_Handsoldering, symbol 0EsseivaN_Lib:MCP9700
- added U7: LD39200, 0EsseivaN_Lib:DFN-6-1EP_3x3mm_Pitch0.95mm, symbol 0EsseivaN_Lib:LD39200
- C1, C7: footprint 0EsseivaN_Lib:CP_Radial_D5.0mm_P2.00mm -> 0EsseivaN_Lib:C_0805_HandSoldering
- P2, P3: value 3V5 -> 3V
- R12: value 22 -> 1k
- R5, R8, R9: value 1K -> 1k
Connections:
- net 3V3: now also X4.1 (P1), X6.1 (P1), C11.1, U6.1 (VDD); no longer R12.2
- net BUZZER: now also X4.2 (P2)
- net GND: now also R12.1, C10.2, C11.2, C9.2, U6.3 (GND), U7.3 (GND), U7.7 (EP)
- net VBAT: now also C9.1, U7.6 (IN)
- net WATER: now also X6.2 (P2)
- net at R11.2: now also R13.2, C10.1, U7.1 (OUT), U7.2 (SENSE)
- net RESET renamed TEMP
- net TEMP: now also U6.2 (VOUT)
- net SET renamed ENABLE
- net ENABLE: now also R12.2, U7.5 (EN)
- no-connect marks 5 -> 1
Other:
- note removed: "Max power : 750mW\nDo not set those\ntrimmer above 8 ohm\nSet the current\nto 300mA"
- moved on the sheet: P2, P3, R11, R13, SC1, X4, X6

Commit message: Update 2
Parts:
- removed R11, R13: 6, Resistors_SMD:R_1206_HandSoldering, symbol 0EsseivaN_Lib:R
- added R11, R13: 10R, 0EsseivaN_Lib:Potentiometer_Trimmer_Bourns_3006P, symbol 0EsseivaN_Lib:Trimmer
- C2: footprint 0EsseivaN_Lib:CP_Radial_D5.0mm_P2.00mm -> 0EsseivaN_Lib:C_0805_HandSoldering
- R10: value 4k7 -> 27k
Connections:
- net at P2.1 (Anode): now also R11.2, R11.3
- net at P3.1 (Anode): now also R13.2, R13.3
- net at C10.1, U7.1 (OUT), U7.2 (SENSE): now also R11.1, R13.1
Other:
- moved on the sheet: P2, P3, V1
Changed lines of the file:
@@
 Sheet 1 1
 Title "Lampe Solaire"
-Date "2019-06-16"
+Date "2019-06-17"
 Rev "6"
 Comp "EsseivaN"
@@
 L 0EsseivaN_Lib:LED P2
 U 1 1 5B69855B
-P 9600 5550
-F 0 "P2" V 9547 5372 60  0000 R CNN
-F 1 "3V" V 9653 5372 60  0000 R CNN
-F 2 "0EsseivaN_Lib:CH_02P" H 9600 5550 60  0001 C CNN
-F 3 "" H 9600 5550 60  0000 C CNN
-	1    9600 5550
+P 9600 5600
+F 0 "P2" V 9547 5422 60  0000 R CNN
+F 1 "3V" V 9653 5422 60  0000 R CNN
+F 2 "0EsseivaN_Lib:CH_02P" H 9600 5600 60  0001 C CNN
+F 3 "" H 9600 5600 60  0000 C CNN
+	1    9600 5600
 	0    1    1    0
 $EndComp
@@
 L 0EsseivaN_Lib:LED P3
 U 1 1 5B69EE95
-P 10000 5550
-F 0 "P3" V 9947 5628 60  0000 L CNN
-F 1 "3V" V 10053 5628 60  0000 L CNN
-F 2 "0EsseivaN_Lib:CH_02P" H 10000 5550 60  0001 C CNN
-F 3 "" H 10000 5550 60  0000 C CNN
-	1    10000 5550
+P 10350 5600
+F 0 "P3" V 10297 5678 60  0000 L CNN
+F 1 "3V" V 10403 5678 60  0000 L CNN
+F 2 "0EsseivaN_Lib:CH_02P" H 10350 5600 60  0001 C CNN
+F 3 "" H 10350 5600 60  0000 C CNN
+	1    10350 5600
 	0    1    1    0
 $EndComp
@@
 Connection ~ 4900 900
 Wire Wire Line
-	5300 900  5300 1500
+	5300 900  5300 1150
 Connection ~ 4500 2000
 Wire Wire Line
@@
 L 0EsseivaN_Lib:GND #PWR032
 U 1 1 5B69BE87
-P 9600 5700
-F 0 "#PWR032" H 9600 5400 50  0001 C CNN
-F 1 "GND" H 9600 5500 50  0001 C CNN
-F 2 "" H 9600 5700 50  0000 C CNN
-F 3 "" H 9600 5700 50  0000 C CNN
-	1    9600 5700
+P 9600 5750
+F 0 "#PWR032" H 9600 5450 50  0001 C CNN
+F 1 "GND" H 9600 5550 50  0001 C CNN
+F 2 "" H 9600 5750 50  0000 C CNN
+F 3 "" H 9600 5750 50  0000 C CNN
+	1    9600 5750
 	1    0    0    -1
 $EndComp
@@
 P 1950 2400
 F 0 "R10" H 1880 2354 50  0000 R CNN
-F 1 "4k7" H 1880 2445 50  0000 R CNN
+F 1 "27k" H 1880 2445 50  0000 R CNN
 F 2 "0EsseivaN_Lib:R_0805_HandSoldering" V 1880 2400 50  0001 C CNN
 F 3 "" H 1950 2400 50  0000 C CNN
@@
 	4900 2000 5300 2000
 Wire Wire Line
-	5300 1900 5300 2000
+	5300 1550 5300 2000
 Connection ~ 5300 2000
 $Comp
@@
 	7400 1400 9800 1400
 Wire Wire Line
-	9600 5650 9600 5700
+	9600 5700 9600 5750
 $Comp
 L 0EsseivaN_Lib:GND #PWR0101
 U 1 1 5C5978CB
-P 10000 5700
-F 0 "#PWR0101" H 10000 5400 50  0001 C CNN
-F 1 "GND" H 10000 5500 50  0001 C CNN
-F 2 "" H 10000 5700 50  0000 C CNN
-F 3 "" H 10000 5700 50  0000 C CNN
-	1    10000 5700
+P 10350 5750
+F 0 "#PWR0101" H 10350 5450 50  0001 C CNN
+F 1 "GND" H 10350 5550 50  0001 C CNN
+F 2 "" H 10350 5750 50  0000 C CNN
+F 3 "" H 10350 5750 50  0000 C CNN
+	1    10350 5750
 	1    0    0    -1
 $EndComp
@@
 L 0EsseivaN_Lib:LiPo V1
 U 1 1 5B6566C3
-P 5300 1700
-F 0 "V1" H 5450 1950 60  0000 C CNN
-F 1 "Li battery" H 5600 1850 60  0000 C CNN
-F 2 "0EsseivaN_Lib:CH_03P" H 5310 1750 60  0001 C CNN
-F 3 "" H 5310 1750 60  0001 C CNN
-F 4 "3V7" H 5500 1550 60  0000 C CNN "Voltage"
-F 5 "3200mAh" H 5300 1700 60  0001 C CNN "Capacity"
-	1    5300 1700
+P 5300 1350
+F 0 "V1" H 5450 1600 60  0000 C CNN
+F 1 "Li battery" H 5600 1500 60  0000 C CNN
+F 2 "0EsseivaN_Lib:CH_03P" H 5310 1400 60  0001 C CNN
+F 3 "" H 5310 1400 60  0001 C CNN
+F 4 "3V7" H 5500 1200 60  0000 C CNN "Voltage"
+F 5 "3200mAh" H 5300 1350 60  0001 C CNN "Capacity"
+	1    5300 1350
 	1    0    0    -1
 $EndComp
@@
 F 0 "C2" V 4650 1500 60  0000 C CNN
 F 1 "10uF" V 4750 1550 60  0000 C CNN
-F 2 "0EsseivaN_Lib:CP_Radial_D5.0mm_P2.00mm" H 4900 1400 60  0001 C CNN
+F 2 "0EsseivaN_Lib:C_0805_HandSoldering" H 4900 1400 60  0001 C CNN
 F 3 "" H 4900 1400 60  0000 C CNN
 	1    4900 1400
@@
 $EndComp
 Wire Wire Line
-	9600 5400 9600 5450
-Wire Wire Line
-	10000 5400 10000 5450
-$Comp
-L 0EsseivaN_Lib:R R11
-U 1 1 5CE208BB
-P 9600 5200
-F 0 "R11" H 9530 5154 50  0000 R CNN
-F 1 "6" H 9530 5245 50  0000 R CNN
-F 2 "Resistors_SMD:R_1206_HandSoldering" V 9530 5200 50  0001 C CNN
-F 3 "" H 9600 5200 50  0000 C CNN
-	1    9600 5200
-	-1   0    0    1
-$EndComp
-$Comp
-L 0EsseivaN_Lib:R R13
-U 1 1 5CE20D21
-P 10000 5200
-F 0 "R13" H 9930 5154 50  0000 R CNN
-F 1 "6" H 9930 5245 50  0000 R CNN
-F 2 "Resistors_SMD:R_1206_HandSoldering" V 9930 5200 50  0001 C CNN
-F 3 "" H 10000 5200 50  0000 C CNN
-	1    10000 5200
-	-1   0    0    1
-$EndComp
+	9600 5450 9600 5500
+Wire Wire Line
+	10350 5450 10350 5500
 Text Label 1050 4050 2    60   ~ 0
 RESET_RF
@@
 NoConn ~ 8150 5100
 Wire Wire Line
-	10000 4950 9600 4950
-Wire Wire Line
 	9600 4950 9600 5000
 Wire Wire Line
-	10000 4950 10000 5000
-Wire Wire Line
-	10000 5650 10000 5700
+	10350 4950 10350 5000
+Wire Wire Line
+	10350 5700 10350 5750
 Wire Wire Line
 	8850 4950 8900 4950
-Connection ~ 9600 4950
 Wire Wire Line
 	8850 5050 8900 5050
@@
 Wire Wire Line
 	7100 5000 7300 5000
+$Comp
+L 0EsseivaN_Lib:Trimmer R11
+U 1 1 5D0C5008
+P 9600 5200
+F 0 "R11" H 9753 5246 50  0000 L CNN
+F 1 "10R" H 9753 5155 50  0000 L CNN
+F 2 "0EsseivaN_Lib:Potentiometer_Trimmer_Bourns_3006P" V 9530 5200 50  0001 C CNN
+F 3 "" H 9600 5200 50  0000 C CNN
+	1    9600 5200
+	1    0    0    -1
+$EndComp
+Wire Wire Line
+	9400 5300 9400 5450
+Wire Wire Line
+	9400 5450 9600 5450
+Wire Wire Line
+	9600 5450 9600 5400
+$Comp
+L 0EsseivaN_Lib:Trimmer R13
+U 1 1 5D0E9359
+P 10350 5200
+F 0 "R13" H 10503 5246 50  0000 L CNN
+F 1 "10R" H 10503 5155 50  0000 L CNN
+F 2 "0EsseivaN_Lib:Potentiometer_Trimmer_Bourns_3006P" V 10280 5200 50  0001 C CNN
+F 3 "" H 10350 5200 50  0000 C CNN
+	1    10350 5200
+	1    0    0    -1
+$EndComp
+Wire Wire Line
+	10150 5300 10100 5300
+Wire Wire Line
+	10100 5300 10100 5450
+Wire Wire Line
+	10100 5450 10350 5450
+Wire Wire Line
+	10350 5450 10350 5400
+Wire Wire Line
+	9600 4950 10350 4950
+Connection ~ 9600 4950
+Connection ~ 9600 5450
+Connection ~ 10350 5450
 $EndSCHEMATC
