File: Hardware/LampeSolaire/LampeSolaire.sch (KiCad schematic (older format))
At the start: 48 parts, among them P1 1V8, P2 3V, P3 3V, P4 2V, T1 SI2333, T2 SI2333, T3 FDN337, U1 MCP73832, U2 MCP121, U3 NCP114ASN330T1G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

Commit message: preparation for v6
Parts:
- removed W2: TEST_2P, 0EsseivaN_Lib:Pin_Header_Straight_1x02_Pitch2.54mm, symbol 0EsseivaN_Lib:TEST_2P
- added C12: 100nF, 0EsseivaN_Lib:C_0805_HandSoldering, symbol 0EsseivaN_Lib:CAPA
- C11, C3, C4, C5, C6, C8, C9: footprint Capacitors_SMD:C_1206_HandSoldering -> 0EsseivaN_Lib:C_0805_HandSoldering
- P4: value 2V -> 1V8
- R12, R8, R9: value 1k -> 4k7
- R5: value 1k -> 100k
- R7: value 100k -> 10M
- X2: footprint 0EsseivaN_Lib:Pin_Header_Straight_1x06_Pitch2.54mm -> 0EsseivaN_Lib:Pin_Header_Straight_1x05_Pitch2.54mm
Connections:
- net 3V3: now also C12.1; no longer R5.2
- net GND: now also R5.1
- net RESET_RF: now also R5.2, C12.2; no longer R5.1
- net VSC: now also SC1.1 (+)
Other:
- moved on the sheet: C7, C8, R5, R7, R8, R9, U4, X6

Commit message: Version 6 final
Parts:
- added R14, R15: NP, 0EsseivaN_Lib:R_0805_HandSoldering, symbol 0EsseivaN_Lib:R
- added U8: RF_RECEIVER, NP, 0EsseivaN_Lib:RF_RECEIVER, symbol 0EsseivaN_Lib:RF_RECEIVER
- C9: value 100nF -> 4.7uF
- P1: footprint 0EsseivaN_Lib:LED_D3.0mm -> 0EsseivaN_Lib:D_0603_HandSoldering
Connections:
- net 3V3: now also U8.2 (VCC)
- net BUZZER: now also U5.17 (RA6); no longer U5.3 (RA4)
- net GND: now also U8.1 (VSS)
- net ICSPCLK: now also U8.7 (VT)
- net ICSPDAT: now also U8.6 (D3)
- net IRQ1: now also U5.10 (RB3); no longer U5.12 (RB5)
- net MISO: now also U8.3 (D0)
- net MOSI: now also U8.4 (D1)
- net SCK: now also U8.5 (D2)
- net TEMP: now also U5.3 (RA4); no longer U5.17 (RA6)
- net WATER: now also U5.12 (RB5); no longer U5.10 (RB3)
- net at P2.2 (Anode), R11.2, R11.3: now also R14.1
- net at P3.2 (Anode), R13.2, R13.3: now also R15.1
- net at C10.1, R11.1, R13.1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: now also R14.2, R15.2
Other:
- moved on the sheet: C10, C9, P2, P3, R11, R12, R13, U7

Commit message: tbd
Parts:
- removed C11, C12: 100nF, 0EsseivaN_Lib:C_0805_HandSoldering, symbol 0EsseivaN_Lib:CAPA
- removed R5: 100k, 0EsseivaN_Lib:R_0805_HandSoldering, symbol 0EsseivaN_Lib:R
- removed R8, R9: 4k7, 0EsseivaN_Lib:R_0805_HandSoldering, symbol 0EsseivaN_Lib:R
- removed U4: MRF89XAM8A, 0EsseivaN_Lib:MRF89XAM8A, symbol 0EsseivaN_Lib:MRF89XAM8A
- removed U6: MCP9700, 0EsseivaN_Lib:SOT-23_Handsoldering, symbol 0EsseivaN_Lib:MCP9700
Connections:
- net TEMP is gone; now on net LED: U5.3 (RA4)
- net ~CSCON is gone; now on net D2: U5.1 (RA2)
- net BUZZER: now also U5.11 (RB4); no longer U5.17 (RA6)
- net ICSPCLK: no longer U8.7 (VT)
- net ICSPDAT: no longer U8.6 (D3)
- net LED: no longer U5.2 (RA3)
- net IRQ0: no longer names the net of U5.7 (RB0)
- net IRQ1: no longer names the net of U5.10 (RB3)
- net MISO: no longer names the net of U5.8 (RB1)
- net MISO: no longer U8.3 (D0)
- net MOSI: no longer names the net of U5.9 (RB2)
- net MOSI: no longer U8.4 (D1)
- net RESET_RF renamed D0
- net D0: now also U8.3 (D0)
- net SCK renamed D2
- net D2: no longer U5.11 (RB4)
- net ~CSDATA renamed D1
- net D1: now also U8.4 (D1)
- new net D3: U5.2 (RA3), U8.6 (D3)
- new net VT: U5.17 (RA6), U8.7 (VT)
- no-connect marks 1 -> 5
Other:
- moved on the sheet: C10, C7, C8, C9, P2, P3, P4, R11, R12, R13, R14, R15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

Commit message: first upgrade for v7
Parts:
- added X1, X3: POWER, symbol 0EsseivaN_Lib:CONN_01X03
- P2, P3, SC1, X4, X6: footprint 0EsseivaN_Lib:CH_02P -> 0EsseivaN_Lib:Pin_Header_Straight_1x02_Pitch2.54mm
- V1: footprint 0EsseivaN_Lib:CH_03P -> 0EsseivaN_Lib:Pin_Header_Straight_1x02_Pitch2.54mm
Connections:
- net 3V3: now also X3.2 (P2)
- net GND: now also X3.3 (P3)
- net GND_ALIM: now also X1.3 (P3)
- net VBAT: now also X3.1 (P1); no longer C4.1, T2.3 (D), U3.1 (VIN)
- net at U3.5 (VOUT), W5.1: now also X1.2 (P2)
- new net VBAT_1: C4.1, T2.3 (D), U3.1 (VIN), X1.1 (P1)
Other:
- moved on the sheet: C1, C2, C3, C4, C5, C6, C7, F1, P1, P4, R1, R10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

Commit message: V7
Parts:
- removed X1, X3: POWER, symbol 0EsseivaN_Lib:CONN_01X03
- added P5, P6, P8: GREEN, 0EsseivaN_Lib:D_0603_HandSoldering, symbol 0EsseivaN_Lib:LED
- added P7: RED, 0EsseivaN_Lib:D_0603_HandSoldering, symbol 0EsseivaN_Lib:LED
- added R16, R8: 270R, 0EsseivaN_Lib:R_0805_HandSoldering, symbol 0EsseivaN_Lib:R
- added R17, R18: 10k, 0EsseivaN_Lib:R_0805_HandSoldering, symbol 0EsseivaN_Lib:R
- added R5: 1k5, 0EsseivaN_Lib:R_0805_HandSoldering, symbol 0EsseivaN_Lib:R
- added R9: 330R, 0EsseivaN_Lib:R_0805_HandSoldering, symbol 0EsseivaN_Lib:R
- added V2: Li battery, 0EsseivaN_Lib:Pin_Header_Straight_1x02_Pitch2.54mm, symbol 0EsseivaN_Lib:CONN_01X02
- added X1: BATTERY_JUMPER, 0EsseivaN_Lib:Pin_Header_Straight_1x02_Pitch2.54mm, symbol 0EsseivaN_Lib:CONN_01X02
- P4: value 1V8 -> RED
- U5: value PIC16F1827 -> PIC16LF1827
- V1: footprint 0EsseivaN_Lib:Pin_Header_Straight_1x02_Pitch2.54mm -> 0EsseivaN_Lib:18650 Battery holder
Connections:
- net VBAT_1 is gone; now on net VBAT: C4.1, T2.3 (D), U3.1 (VIN)
- net 3V3: now also R16.2, R5.2, R8.2, R9.2
- net D0: now also U5.20 (RA1); no longer U5.19 (RA0)
- net D1: now also U5.17 (RA6); no longer U5.20 (RA1)
- net D2: now also U5.18 (RA7); no longer U5.1 (RA2)
- net D3: now also U5.19 (RA0); no longer U5.2 (RA3)
- net ENABLE: now also U5.10 (RB3); no longer U5.18 (RA7)
- net GND: now also P5.1 (Cathode), R18.1
- net GND_ALIM: now also V2.2 (P2)
- net VBAT: now also R17.2
- net VT: now also U5.12 (RB5); no longer U5.17 (RA6)
- net WATER: now also U5.3 (RA4); no longer U5.12 (RB5)
- net at C2.1, F1.2, V1.1 (V+)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: now also V2.1 (P1)
- net LED_G: now reaches U5.7 (RB0)
- net LED_G: now also P4.1 (Cathode)
- net LED_R: now reaches U5.8 (RB1)
- net LED_R: now also P6.1 (Cathode)
- net BATTERY_LVL: now reaches U5.9 (RB2)
- net BATTERY_LVL: now also X1.2 (P2)
- removed net LED: P4.1 (Cathode), U5.3 (RA4)
- new net: R17.1, R18.2, X1.1 (P1)
- new net: P7.2 (Anode), R9.1
- new net: P8.2 (Anode), R16.1
- new net: P6.2 (Anode), R8.1
- new net: P5.2 (Anode), R5.1
- new net BATTERY_IND_G: P8.1 (Cathode), U5.1 (RA2)
- new net BATTERY_IND_R: P7.1 (Cathode), U5.2 (RA3)
- no-connect marks 5 -> 1
Other:
- moved on the sheet: C10, C3, C4, C5, C7, C8, C9, F1, P2, P3, P4, R11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
