File: Hardware/LampeSolaire/LampeSolaire.kicad_pcb (KiCad board)
At the start: 2 copper layers, 83 x 64 mm, 50 parts, among them P1 1V8, P2 3V, P3 3V, P4 2V, T1 SI2333, T2 SI2333, T3 FDN337, U1 MCP73832, U2 MCP121, U3 NCP114ASN330T1G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

Commit message: Update 2
Parts:
- C2: footprint 0EsseivaN_Lib:CP_Radial_D5.0mm_P2.00mm -> 0EsseivaN_Lib:C_0805_HandSoldering
- R10: value 4k7 -> 27k
- R11, R13: value 6 -> 10R; footprint Resistors_SMD:R_1206_HandSoldering -> 0EsseivaN_Lib:Potentiometer_Trimmer_Bourns_3006P; moved to F.Cu
- moved P2 16.3 mm to (77.6, 111.4)
- moved P3 16.3 mm to (86.5, 111.4)
- moved R11 15.7 mm to (105.6, 100.0), turned to 90 degrees
- moved R13 4.02 mm to (98.0, 100.0), turned to 90 degrees
- moved C2 1.80 mm to (91.1, 56.8)
- moved C9 0.42 mm to (85.3, 96.2)
Connections:
- R11 pad 1: Net-(P2-Pad1) -> Net-(C10-Pad1)
- R11 pad 2: Net-(C10-Pad1) -> Net-(P2-Pad1)
- R13 pad 1: Net-(P3-Pad1) -> Net-(C10-Pad1)
- R13 pad 2: Net-(C10-Pad1) -> Net-(P3-Pad1)
Routing:
- net Net-(P2-Pad1): track 9.15 -> 38.9 mm
- net Net-(P3-Pad1): track 9.15 -> 20.1 mm
- net GND: track 242.3 -> 251.6 mm, vias 13 -> 11
- net Net-(C10-Pad1): track 43.8 -> 41.0 mm, vias 3 -> 1
- added copper zone on F.Cu, net VSC
Other:
- board size 83 x 64 mm -> 83 x 74 mm
- board text added: "Lampe Solaire 18.06.19 - V6 EsseivaN"
- board text removed: "Lampe Solaire 15.06.19 - V6 EsseivaN"

Commit message: preparation for v6
Parts:
- removed W2: TEST_2P, 0EsseivaN_Lib:Pin_Header_Straight_1x02_Pitch2.54mm
- added C12: 100nF, 0EsseivaN_Lib:C_0805_HandSoldering, B.Cu at (102.5, 79.7)
- C11, C3, C4, C5, C6, C8, C9: footprint Capacitors_SMD:C_1206_HandSoldering -> 0EsseivaN_Lib:C_0805_HandSoldering
- P4: value 2V -> 1V8
- R12, R8, R9: value 1k -> 4k7
- R5: value 1k -> 100k
- R7: value 100k -> 10M
- X2: footprint 0EsseivaN_Lib:Pin_Header_Straight_1x06_Pitch2.54mm -> 0EsseivaN_Lib:Pin_Header_Straight_1x05_Pitch2.54mm
- moved C10 1.30 mm to (73.3, 94.9)
- moved C3 1.27 mm to (96.2, 50.5)
- moved C4 1.27 mm to (119.0, 58.1)
- moved C9 0.76 mm to (86.0, 96.2)
- moved C11 0.70 mm to (67.0, 63.2)
- moved C5 0.54 mm to (119.0, 58.1)
Connections:
- R5 pad 1: /RESET_RF -> GND
- R5 pad 2: 3V3 -> /RESET_RF
- SC1 pad 1: Net-(SC1-Pad1) -> VSC
Routing:
- net /RESET_RF: track 38.2 -> 45.7 mm, vias 1 -> 2
- net Net-(SC1-Pad1): track 6.21 -> 0.00 mm
- net VSC: track 33.3 -> 27.5 mm
- net GND: track 251.6 -> 247.6 mm
- net VBAT: track 86.7 -> 90.1 mm
- net 3V3: track 181.2 -> 184.1 mm
- net Net-(C10-Pad1): track 41.0 -> 42.9 mm

Commit message: Version 6 final
Parts:
- added R14: NP, 0EsseivaN_Lib:R_0805_HandSoldering, F.Cu at (81.0, 103.8)
- added R15: NP, 0EsseivaN_Lib:R_0805_HandSoldering, F.Cu at (83.5, 103.8)
- added U8: RF_RECEIVER, NP, 0EsseivaN_Lib:RF_RECEIVER, F.Cu at (51.7, 79.7)
- C9: value 100nF -> 4.7uF
- P1: footprint 0EsseivaN_Lib:LED_D3.0mm -> 0EsseivaN_Lib:D_0603_HandSoldering; moved to B.Cu
- turned P1 to 0 degrees
- turned P4 to 180 degrees
Connections:
- P1 pad 1: VSC -> Net-(P1-Pad1)
- P1 pad 2: Net-(P1-Pad2) -> VSC
- P2 pad 1: Net-(P2-Pad1) -> GND
- P2 pad 2: GND -> Net-(P2-Pad2)
- P3 pad 1: Net-(P3-Pad1) -> GND
- P3 pad 2: GND -> Net-(P3-Pad2)
- P4 pad 1: Net-(P4-Pad1) -> /LED
- P4 pad 2: /LED -> Net-(P4-Pad2)
- R1 pad 2: Net-(P1-Pad2) -> Net-(P1-Pad1)
- R11 pad 2: Net-(P2-Pad1) -> Net-(P2-Pad2)
- R11 pad 3: Net-(P2-Pad1) -> Net-(P2-Pad2)
- R13 pad 2: Net-(P3-Pad1) -> Net-(P3-Pad2)
- R13 pad 3: Net-(P3-Pad1) -> Net-(P3-Pad2)
- R6 pad 1: Net-(P4-Pad1) -> Net-(P4-Pad2)
- U5 pad 10: /WATER -> /IRQ1
- U5 pad 12: /IRQ1 -> /WATER
- U5 pad 17: /TEMP -> /BUZZER
- U5 pad 3: /BUZZER -> /TEMP
Routing:
- net /SCK: track 32.5 -> 83.5 mm, vias 4 -> 7
- net Net-(P2-Pad2): track 0.00 -> 40.4 mm, vias 0 -> 1
- net Net-(P2-Pad1): track 38.9 -> 0.00 mm, vias 1 -> 0
- net /MISO: track 42.8 -> 70.9 mm, vias 2 -> 4
- net GND: track 247.6 -> 273.6 mm, vias 11 -> 13
- net /WATER: track 58.4 -> 33.0 mm, vias 5 -> 3
- net /MOSI: track 52.1 -> 77.3 mm, vias 6 -> 8
- net Net-(P3-Pad2): track 0.00 -> 24.9 mm, vias 0 -> 2
- net Net-(P3-Pad1): track 20.1 -> 0.00 mm, vias 1 -> 0
- net 3V3: track 184.1 -> 198.1 mm, vias 19 -> 21
- net /TEMP: track 32.6 -> 19.4 mm, vias 4 -> 2
- net /ICSPDAT: track 44.9 -> 56.1 mm, vias 4 -> 5
- net /ICSPCLK: track 46.7 -> 57.6 mm
- net /BUZZER: track 24.4 -> 15.1 mm
- net /IRQ1: track 33.9 -> 42.7 mm, vias 4 -> 2
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- added copper zone on F.Cu, net /VBAT_0
Other:
- board size 83 x 74 mm -> 92 x 74 mm
- board text added: "B.Cu - V6.2"
- board text added: "B.Mask - V6.2"
- board text added: "F.Cu - V6.2"
- board text added: "F.Mask - V6.2"
- board text added: "For P2"
- board text added: "For P3"
- board text added: "Lampe Solaire 24.06.19 - V6.2 EsseivaN"
- board text added: "NP"
- board text added: "Solar Panel Charger Power Supply"
- board text removed: "B.Cu - V6"
- board text removed: "B.Mask - V6"
- board text removed: "F.Cu - V6"
- board text removed: "F.Mask - V6"
- board text removed: "Lampe Solaire 18.06.19 - V6 EsseivaN"

Commit message: Software update
Parts:
- P1: moved to F.Cu
- turned P4 to 0 degrees
Routing:
- net VSC: track 28.6 -> 29.1 mm, vias 1 -> 2
- net Net-(P1-Pad1): vias 0 -> 1

Commit message: first upgrade for v7
Parts:
- removed C11, C12: 100nF, 0EsseivaN_Lib:C_0805_HandSoldering
- removed the PERC-4.5mm at (135.1, 100.0)
- removed R5: 100k, 0EsseivaN_Lib:R_0805_HandSoldering
- removed R8, R9: 4k7, 0EsseivaN_Lib:R_0805_HandSoldering
- removed U4: MRF89XAM8A, 0EsseivaN_Lib:MRF89XAM8A
- removed U6: MCP9700, 0EsseivaN_Lib:SOT-23_Handsoldering
- added REF**: BoardCutter_1, 0EsseivaN_Lib:BoardCutter_1, F.Cu at (140.7, 59.7)
- added REF**: BoardCutter_10, 0EsseivaN_Lib:BoardCutter_10, F.Cu at (57.5, 59.7)
- added REF**: BoardCutter_2, 0EsseivaN_Lib:BoardCutter_2, F.Cu at (139.3, 59.7)
- added REF**: BoardCutter_10, 0EsseivaN_Lib:BoardCutter_10, F.Cu at (128.6, 59.7)
- added REF**: BoardCutter_10, 0EsseivaN_Lib:BoardCutter_10, F.Cu at (118.5, 59.7)
- added REF**: BoardCutter_10, 0EsseivaN_Lib:BoardCutter_10, F.Cu at (108.3, 59.7)
- added REF**: BoardCutter_10, 0EsseivaN_Lib:BoardCutter_10, F.Cu at (98.1, 59.7)
- added REF**: BoardCutter_10, 0EsseivaN_Lib:BoardCutter_10, F.Cu at (88.0, 59.7)
- added REF**: BoardCutter_10, 0EsseivaN_Lib:BoardCutter_10, F.Cu at (77.8, 59.7)
- added REF**: BoardCutter_10, 0EsseivaN_Lib:BoardCutter_10, F.Cu at (67.7, 59.7)
- added W4: TEST_2P, 0EsseivaN_Lib:Pin_Header_Straight_1x02_Pitch2.54mm, F.Cu at (133.7, 65.5)
- added W4: TEST_2P, 0EsseivaN_Lib:Pin_Header_Straight_1x02_Pitch2.54mm, F.Cu at (129.9, 65.5)
- added W4: TEST_2P, 0EsseivaN_Lib:Pin_Header_Straight_1x02_Pitch2.54mm, F.Cu at (126.1, 65.5)
- C1, C4, F1, R3, R4, T2, T3, U2, U3: moved to F.Cu
- P2, P3, SC1, X4, X6: footprint 0EsseivaN_Lib:CH_02P -> 0EsseivaN_Lib:Pin_Header_Straight_1x02_Pitch2.54mm
- V1: footprint 0EsseivaN_Lib:CH_03P -> 0EsseivaN_Lib:Pin_Header_Straight_1x02_Pitch2.54mm
- moved U8 73.7 mm to (125.4, 81.0), turned to 90 degrees
- moved C3 18.9 mm to (114.7, 54.7), turned to 0 degrees
- moved W5 18.4 mm to (129.9, 51.5), turned to 0 degrees
- moved V1 18.4 mm to (88.0, 52.1), turned to 0 degrees
- moved U2 17.2 mm to (114.7, 51.5)
- moved T2 16.8 mm to (105.1, 54.0), turned to 0 degrees
- moved R3 15.4 mm to (110.2, 51.5), turned to 270 degrees
- moved P1 11.5 mm to (72.1, 48.9)
- moved SC1 9.49 mm to (62.6, 52.1), turned to 0 degrees
- moved R1 9.00 mm to (68.3, 52.1), turned to 90 degrees
- moved F1 8.68 mm to (96.2, 48.9)
- moved U3 8.31 mm to (121.0, 53.4)
- moved C5 7.47 mm to (117.8, 65.5), turned to 180 degrees
- moved W3 7.06 mm to (81.0, 52.1)
- moved T1 6.24 mm to (96.2, 54.0), turned to 0 degrees
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Connections:
- C4 pad 1: VBAT -> /VBAT_1
- T2 pad 3: VBAT -> /VBAT_1
- U3 pad 1: VBAT -> /VBAT_1
- U5 pad 1: /~CSCON -> /D2
- U5 pad 10: /IRQ1 -> Net-(U5-Pad10)
- U5 pad 11: /SCK -> /BUZZER
- U5 pad 17: /BUZZER -> /VT
- U5 pad 19: /RESET_RF -> /D0
- U5 pad 2: /LED -> /D3
- U5 pad 20: /~CSDATA -> /D1
- U5 pad 3: /TEMP -> /LED
- U5 pad 7: /IRQ0 -> Net-(U5-Pad7)
- U5 pad 8: /MISO -> Net-(U5-Pad8)
- U5 pad 9: /MOSI -> Net-(U5-Pad9)
- U8 pad 3: /MISO -> /D0
- U8 pad 4: /MOSI -> /D1
- U8 pad 5: /SCK -> /D2
- U8 pad 6: /ICSPDAT -> /D3
- U8 pad 7: /ICSPCLK -> /VT
Routing:
- net 3V3: track 198.1 -> 56.3 mm, vias 21 -> 6
- net GND: track 273.6 -> 135.4 mm, vias 13 -> 5
- net /SCK: track 83.5 -> 0.00 mm, vias 7 -> 0
- net VBAT: track 89.5 -> 8.22 mm, vias 3 -> 1
- net /MOSI: track 77.3 -> 0.00 mm, vias 8 -> 0
- net /MISO: track 70.9 -> 0.00 mm, vias 4 -> 0
- net /IRQ0: track 58.5 -> 0.00 mm, vias 6 -> 0
- net /ICSPCLK: track 57.6 -> 0.00 mm, vias 4 -> 0
- net /ICSPDAT: track 56.1 -> 0.00 mm, vias 5 -> 0
- net /~CSCON: track 48.7 -> 0.00 mm, vias 1 -> 0
- net /RESET_RF: track 43.8 -> 0.00 mm, vias 1 -> 0
- net /IRQ1: track 42.7 -> 0.00 mm, vias 2 -> 0
- net /~CSDATA: track 41.2 -> 0.00 mm, vias 4 -> 0
- net /~RST: track 39.3 -> 7.19 mm, vias 2 -> 0
- net Net-(R4-Pad1): track 38.6 -> 7.54 mm, vias 2 -> 0
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- removed copper zone on F.Cu, net /VBAT_0
- removed copper zone on B.Cu, net 3V3
- removed copper zone on F.Cu, net GND
- removed copper zone on B.Cu, net GND_ALIM
- removed copper zone on F.Cu, net VSC
Other:
- outline, holes or cut-outs redrawn

Commit message: V7
Parts:
- removed REF**: BoardCutter_1, 0EsseivaN_Lib:BoardCutter_1
- removed REF** (x8): BoardCutter_10, 0EsseivaN_Lib:BoardCutter_10
- removed REF**: BoardCutter_2, 0EsseivaN_Lib:BoardCutter_2
- removed the W4 at (133.7, 65.5)
- removed the W4 at (129.9, 65.5)
- removed the W4 at (126.1, 65.5)
- removed the W4 at (126.1, 51.5)
- added P5: GREEN, 0EsseivaN_Lib:D_0603_HandSoldering, F.Cu at (132.4, 80.1)
- added P6: GREEN, 0EsseivaN_Lib:D_0603_HandSoldering, F.Cu at (107.7, 113.1)
- added P7: RED, 0EsseivaN_Lib:D_0603_HandSoldering, F.Cu at (93.1, 94.0)
- added P8: GREEN, 0EsseivaN_Lib:D_0603_HandSoldering, F.Cu at (88.0, 94.0)
- added PERC-4.5mm: ~, 0EsseivaN_Lib:PERC-4.5mm, F.Cu at (135.1, 100.0)
- added R16: 270R, 0EsseivaN_Lib:R_0805_HandSoldering, F.Cu at (85.4, 94.0)
- added R17: 10k, 0EsseivaN_Lib:R_0805_HandSoldering, F.Cu at (122.3, 80.1)
- added R18: 10k, 0EsseivaN_Lib:R_0805_HandSoldering, F.Cu at (117.2, 80.1)
- added R5: 1k5, 0EsseivaN_Lib:R_0805_HandSoldering, F.Cu at (129.9, 80.1)
- added R8: 270R, 0EsseivaN_Lib:R_0805_HandSoldering, F.Cu at (110.2, 110.5)
- added R9: 330R, 0EsseivaN_Lib:R_0805_HandSoldering, F.Cu at (90.5, 94.0)
- added V2: Li battery, 0EsseivaN_Lib:Pin_Header_Straight_1x02_Pitch2.54mm, F.Cu at (88.0, 52.1)
- added W4: TEST_2P, 0EsseivaN_Lib:Pin_Header_Straight_1x02_Pitch2.54mm, F.Cu at (127.3, 51.5)
- added X1: BATTERY_JUMPER, 0EsseivaN_Lib:Pin_Header_Straight_1x02_Pitch2.54mm, F.Cu at (100.7, 87.7)
- C6, C7, C8, R1, R10, R6, R7: moved to F.Cu
- P4: value 1V8 -> RED
- U5: value PIC16F1827 -> PIC16LF1827
- V1: footprint 0EsseivaN_Lib:Pin_Header_Straight_1x02_Pitch2.54mm -> 0EsseivaN_Lib:18650 Battery holder
- moved U8 54.3 mm to (93.1, 124.5), turned to 180 degrees
- moved R10 48.5 mm to (98.1, 113.7)
- moved R6 47.3 mm to (110.2, 118.2), turned to 0 degrees
- moved P4 43.7 mm to (107.7, 115.6)
- moved R14 42.5 mm to (122.9, 97.2), turned to 180 degrees
- moved R15 39.4 mm to (122.9, 103.6), turned to 180 degrees
- moved P2 37.9 mm to (112.7, 97.2), turned to 90 degrees
- moved C6 37.3 mm to (89.9, 113.1), turned to 0 degrees
- moved C10 35.7 mm to (107.7, 104.8), turned to 90 degrees
- moved U5 29.1 mm to (89.9, 106.1), turned to 180 degrees
- moved C7 28.5 mm to (99.4, 118.2)
- moved P3 27.4 mm to (112.7, 103.6), turned to 90 degrees
- moved R7 25.7 mm to (96.2, 93.4), turned to 270 degrees
- moved X2 25.5 mm to (65.1, 112.4), turned to 0 degrees
- moved U7 25.5 mm to (104.5, 101.0), turned to 90 degrees
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Connections:
- C4 pad 1: /VBAT_1 -> VBAT
- P4 pad 1: /LED -> /LED_G
- T2 pad 3: /VBAT_1 -> VBAT
- U3 pad 1: /VBAT_1 -> VBAT
- U5 pad 1: /D2 -> /BATTERY_IND_G
- U5 pad 10: Net-(U5-Pad10) -> /ENABLE
- U5 pad 12: /WATER -> /VT
- U5 pad 17: /VT -> /D1
- U5 pad 18: /ENABLE -> /D2
- U5 pad 19: /D0 -> /D3
- U5 pad 2: /D3 -> /BATTERY_IND_R
- U5 pad 20: /D1 -> /D0
- U5 pad 3: /LED -> /WATER
- U5 pad 7: Net-(U5-Pad7) -> /LED_G
- U5 pad 8: Net-(U5-Pad8) -> /LED_R
- U5 pad 9: Net-(U5-Pad9) -> /BATTERY_LVL
Routing:
- net 3V3: track 56.3 -> 223.9 mm, vias 6 -> 11
- net GND_ALIM: track 93.1 -> 214.3 mm
- net VBAT: track 8.22 -> 124.6 mm, vias 1 -> 3
- net GND: track 135.4 -> 204.6 mm, vias 5 -> 6
- net Net-(C2-Pad1): track 13.9 -> 76.0 mm
- net /VPP: track 0.00 -> 43.6 mm, vias 0 -> 2
- net /ICSPCLK: track 0.00 -> 39.5 mm, vias 0 -> 2
- net /ICSPDAT: track 0.00 -> 36.2 mm, vias 0 -> 2
- net /D1: track 0.00 -> 36.0 mm, vias 0 -> 3
- net /VT: track 0.00 -> 33.8 mm, vias 0 -> 3
- net /D2: track 0.00 -> 31.9 mm, vias 0 -> 3
- net /D3: track 0.00 -> 26.9 mm, vias 0 -> 3
- net /D0: track 5.54 -> 32.2 mm, vias 0 -> 3
- net Net-(R17-Pad1): track 0.00 -> 26.7 mm, vias 0 -> 2
- net /LED_G: track 0.00 -> 23.6 mm, vias 0 -> 2
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- added copper zone on F.Cu, net 3V3
- added copper zone on B.Cu, net GND_ALIM
- added copper zone on F.Cu, net VSC
Other:
- board size 92 x 74 mm -> 85 x 83 mm
- board text added: "+"
- board text added: "-"
- board text added: "B.Cu - V7"
- board text added: "B.Mask - V7"
- board text added: "F.Cu - V7"
- board text added: "F.Mask - V7"
- board text added: "IP2"
- board text added: "IP3"
- board text added: "Lampe Solaire 11.08.19 - V7 EsseivaN"
- board text removed: "B.Cu - V6.2"
- board text removed: "B.Mask - V6.2"
- board text removed: "F.Cu - V6.2"
- board text removed: "F.Mask - V6.2"
- board text removed: "For P2"
- board text removed: "For P3"
- board text removed: "Lampe Solaire 24.06.19 - V6.2 EsseivaN"
- board text removed: "Solar Panel Charger Power Supply"

Commit message: Waiting for last check
Parts:
- moved P8 43.1 mm to (119.7, 123.2)
- moved P7 37.9 mm to (117.2, 123.2)
- moved R16 36.1 mm to (113.4, 116.9), turned to 180 degrees
- moved R9 34.2 mm to (113.4, 119.4), turned to 180 degrees
- moved P4 22.3 mm to (128.6, 123.2), turned to 90 degrees
- moved P6 21.0 mm to (126.1, 123.2), turned to 90 degrees
- moved R6 18.4 mm to (128.6, 118.2), turned to 90 degrees
- moved R8 17.6 mm to (126.1, 118.2), turned to 90 degrees
Routing:
- net /LED_G: track 23.6 -> 57.2 mm, vias 2 -> 4
- net /LED_R: track 22.4 -> 53.3 mm, vias 2 -> 5
- net /BATTERY_IND_G: track 17.7 -> 42.6 mm, vias 0 -> 2
- net /BATTERY_IND_R: track 15.7 -> 38.0 mm, vias 0 -> 2
- net 3V3: track 223.9 -> 232.7 mm, vias 11 -> 9
- net Net-(P8-Pad2): track 2.63 -> 9.63 mm
- net Net-(P7-Pad2): track 2.63 -> 4.70 mm
Other:
- board text added: "%"
